File: Circuits/light_gate/light_gate.kicad_pcb (KiCad board)
At the start: 2 copper layers, 38.1 x 20.3 mm, 11 parts, among them J1 Conn_01x03, J2 Conn_01x02, Q1 BC547

Commit message: udated footprints npn
Parts:
- D1: value IRE -> CQY99
- D2: value IRR -> SFH203FA
- Q1: footprint Package_TO_SOT_THT:TO-92_Inline -> Package_TO_SOT_THT:TO-92L_Inline_Wide
- moved Q1 0.87 mm to (145.0, 98.2)
Routing:
- net Net-(D3-Pad2): track 6.13 -> 4.34 mm
- net Net-(Q1-Pad1): track 8.67 -> 9.25 mm
Changed lines of the file:
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@@
       (effects (font (size 1 1) (thickness 0.15)))
     )
-    (fp_text value "IRE" (at 1.27 3.96 90) (layer "F.SilkS")
+    (fp_text value "CQY99" (at 1.27 3.96 90) (layer "F.SilkS")
       (effects (font (size 1 1) (thickness 0.15)))
     )
@@
     )
   )
-  (footprint "Package_TO_SOT_THT:TO-92_Inline" (layer "F.Cu")
-    (at 144.78 99.06 -90)
-    (descr "TO-92 leads in-line, narrow, oval pads, drill 0.75mm (see NXP sot054_po.pdf)")
-    (tags "to-92 sc-43 sc-43a sot54 PA33 transistor")
-    (property "Sheetfile" "light_gate.kicad_sch")
-    (property "Sheetname" "")
-    (attr through_hole)
-    (fp_text reference "Q1" (at 1.27 -3.56 90) (layer "F.SilkS")
-      (effects (font (size 1 1) (thickness 0.15)))
-    )
-    (fp_text value "BC547" (at 1.27 2.79 90) (layer "F.Fab")
-      (effects (font (size 1 1) (thickness 0.15)))
-    )
-    (fp_text user "${REFERENCE}" (at 1.27 0 90) (layer "F.Fab")
-      (effects (font (size 1 1) (thickness 0.15)))
-    )
-    (fp_line (start -0.53 1.85) (end 3.07 1.85) (layer "F.SilkS") (width 0.12))
-    (fp_arc (start 1.27 -2.6) (mid 3.672087 -0.994977) (end 3.108478 1.838478) (layer "F.SilkS") (width 0.12))
-    (fp_arc (start -0.568478 1.838478) (mid -1.132087 -0.994977) (end 1.27 -2.6) (layer "F.SilkS") (width 0.12))
-    (fp_line (start 4 2.01) (end 4 -2.73) (layer "F.CrtYd") (width 0.05))
-    (fp_line (start 4 2.01) (end -1.46 2.01) (layer "F.CrtYd") (width 0.05))
-    (fp_line (start -1.46 -2.73) (end 4 -2.73) (layer "F.CrtYd") (width 0.05))
-    (fp_line (start -1.46 -2.73) (end -1.46 2.01) (layer "F.CrtYd") (width 0.05))
-    (fp_line (start -0.5 1.75) (end 3 1.75) (layer "F.Fab") (width 0.1))
-    (fp_arc (start 1.27 -2.48) (mid 3.561221 -0.949055) (end 3.023625 1.753625) (layer "F.Fab") (width 0.1))
-    (fp_arc (start -0.483625 1.753625) (mid -1.021221 -0.949055) (end 1.27 -2.48) (layer "F.Fab") (width 0.1))
-    (pad "1" thru_hole rect (at 0 0 270) (size 1.05 1.5) (drill 0.75) (layers *.Cu *.Mask)
+  (footprint "Package_TO_SOT_THT:TO-92L_Inline_Wide" (layer "F.Cu")
+    (at 145.012528 98.216694 -90)
+    (descr "TO-92L leads in-line (large body variant of TO-92), also known as TO-226, wide, drill 0.75mm (see https://www.diodes.com/assets/Package-Files/TO92L.pdf and http://www.ti.com/lit/an/snoa059/snoa059.pdf)")
+    (tags "TO-92L Inline Wide transistor")
+    (property "Sheetfile" "light_gate.kicad_sch")
+    (property "Sheetname" "")
+    (attr through_hole)
+    (fp_text reference "Q1" (at 2.54 -3.56 -90) (layer "F.SilkS")
+      (effects (font (size 1 1) (thickness 0.15)))
+    )
+    (fp_text value "BC547" (at 2.54 2.79 -90) (layer "F.Fab")
+      (effects (font (size 1 1) (thickness 0.15)))
+    )
+    (fp_text user "${REFERENCE}" (at 2.54 0 -90) (layer "F.Fab")
+      (effects (font (size 1 1) (thickness 0.15)))
+    )
+    (fp_line (start 0.6 1.7) (end 4.45 1.7) (layer "F.SilkS") (width 0.12))
+    (fp_arc (start 0.1836 -1.098807) (mid 1.143021 -2.192817) (end 2.54 -2.6) (layer "F.SilkS") (width 0.12))
+    (fp_arc (start 2.54 -2.6) (mid 3.936979 -2.192818) (end 4.8964 -1.098807) (layer "F.SilkS") (width 0.12))
+    (fp_arc (start 4.842383 1.112264) (mid 4.666594 1.419753) (end 4.45 1.7) (layer "F.SilkS") (width 0.12))
+    (fp_arc (start 0.6 1.7) (mid 0.389183 1.423933) (end 0.217369 1.122045) (layer "F.SilkS") (width 0.12))
+    (fp_line (start -1 -2.75) (end -1 1.85) (layer "F.CrtYd") (width 0.05))
+    (fp_line (start 6.1 1.85) (end -1 1.85) (layer "F.CrtYd") (width 0.05))
+    (fp_line (start -1 -2.75) (end 6.1 -2.75) (layer "F.CrtYd") (width 0.05))
+    (fp_line (start 6.1 1.85) (end 6.1 -2.75) (layer "F.CrtYd") (width 0.05))
+    (fp_line (start 0.65 1.6) (end 4.4 1.6) (layer "F.Fab") (width 0.1))
+    (fp_arc (start 2.54 -2.48) (mid 4.787211 -1.049019) (end 4.441103 1.592547) (layer "F.Fab") (width 0.1))
+    (fp_arc (start 0.647182 1.602385) (mid 0.290076 -1.043188) (end 2.54 -2.48) (layer "F.Fab") (width 0.1))
+    (pad "1" thru_hole rect (at 0 0 270) (size 1.5 1.5) (drill 0.8) (layers *.Cu *.Mask)
       (net 5 "Net-(Q1-Pad1)") (pinfunction "C") (pintype "passive"))
-    (pad "2" thru_hole oval (at 1.27 0 270) (size 1.05 1.5) (drill 0.75) (layers *.Cu *.Mask)
+    (pad "2" thru_hole circle (at 2.54 0 270) (size 1.5 1.5) (drill 0.8) (layers *.Cu *.Mask)
       (net 3 "Net-(D2-Pad2)") (pinfunction "B") (pintype "input"))
-    (pad "3" thru_hole oval (at 2.54 0 270) (size 1.05 1.5) (drill 0.75) (layers *.Cu *.Mask)
+    (pad "3" thru_hole circle (at 5.08 0 270) (size 1.5 1.5) (drill 0.8) (layers *.Cu *.Mask)
       (net 6 "Net-(D3-Pad2)") (pinfunction "E") (pintype "passive"))
-    (model "${KICAD6_3DMODEL_DIR}/Package_TO_SOT_THT.3dshapes/TO-92_Inline.wrl"
+    (model "${KICAD6_3DMODEL_DIR}/Package_TO_SOT_THT.3dshapes/TO-92L_Inline_Wide.wrl"
       (offset (xyz 0 0 0))
       (scale (xyz 1 1 1))
@@
       (effects (font (size 1 1) (thickness 0.15)))
     )
-    (fp_text value "IRR" (at 1.27 3.96 90) (layer "F.SilkS")
+    (fp_text value "SFH203FA" (at 1.27 3.96 90) (layer "F.SilkS")
       (effects (font (size 1 1) (thickness 0.15)))
     )
@@
   (segment (start 125.73 101.6) (end 127 102.87) (width 0.25) (layer "B.Cu") (net 2))
   (segment (start 127 102.87) (end 127 106.68) (width 0.25) (layer "B.Cu") (net 2))
-  (segment (start 134.62 104.14) (end 129.54 104.14) (width 0.25) (layer "B.Cu") (net 3))
+  (segment (start 121.92 101.6) (end 121.92 99.06) (width 0.25) (layer "B.Cu") (net 3))
+  (segment (start 139.7 101.6) (end 140.543306 100.756694) (width 0.25) (layer "B.Cu") (net 3))
+  (segment (start 118.675 101.585) (end 121.905 101.585) (width 0.25) (layer "B.Cu") (net 3))
   (segment (start 132.08 101.6) (end 132.08 106.68) (width 0.25) (layer "B.Cu") (net 3))
-  (segment (start 140.97 100.33) (end 144.78 100.33) (width 0.25) (layer "B.Cu") (net 3))
-  (segment (start 121.92 101.6) (end 121.905 101.585) (width 0.25) (layer "B.Cu") (net 3))
-  (segment (start 139.7 101.6) (end 140.97 100.33) (width 0.25) (layer "B.Cu") (net 3))
+  (segment (start 129.54 99.06) (end 129.54 104.14) (width 0.25) (layer "B.Cu") (net 3))
+  (segment (start 121.905 101.585) (end 121.92 101.6) (width 0.25) (layer "B.Cu") (net 3))
+  (segment (start 121.92 99.06) (end 129.54 99.06) (width 0.25) (layer "B.Cu") (net 3))
+  (segment (start 132.08 106.68) (end 137.16 106.68) (width 0.25) (layer "B.Cu") (net 3))
   (segment (start 139.7 104.14) (end 139.7 101.6) (width 0.25) (layer "B.Cu") (net 3))
-  (segment (start 121.92 99.06) (end 121.92 101.6) (width 0.25) (layer "B.Cu") (net 3))
-  (segment (start 129.54 99.06) (end 121.92 99.06) (width 0.25) (layer "B.Cu") (net 3))
-  (segment (start 129.54 104.14) (end 129.54 99.06) (width 0.25) (layer "B.Cu") (net 3))
-  (segment (start 132.08 106.68) (end 137.16 106.68) (width 0.25) (layer "B.Cu") (net 3))
-  (segment (start 134.62 104.14) (end 139.7 104.14) (width 0.25) (layer "B.Cu") (net 3))
-  (segment (start 121.905 101.585) (end 118.675 101.585) (width 0.25) (layer "B.Cu") (net 3))
+  (segment (start 140.543306 100.756694) (end 145.012528 100.756694) (width 0.25) (layer "B.Cu") (net 3))
+  (segment (start 129.54 104.14) (end 139.7 104.14) (width 0.25) (layer "B.Cu") (net 3))
   (segment (start 132.08 93.98) (end 137.16 93.98) (width 0.25) (layer "B.Cu") (net 4))
   (segment (start 119.38 93.98) (end 125.73 93.98) (width 0.25) (layer "B.Cu") (net 4))
@@
   (segment (start 142.24 93.98) (end 137.16 93.98) (width 0.25) (layer "B.Cu") (net 4))
   (segment (start 118.675 99.045) (end 118.675 94.685) (width 0.25) (layer "B.Cu") (net 4))
-  (segment (start 137.16 101.6) (end 139.7 99.06) (width 0.25) (layer "B.Cu") (net 5))
-  (segment (start 139.7 99.06) (end 144.78 99.06) (width 0.25) (layer "B.Cu") (net 5))
-  (segment (start 144.78 104.14) (end 147.32 106.68) (width 0.25) (layer "B.Cu") (net 6))
-  (segment (start 144.78 101.6) (end 144.78 104.14) (width 0.25) (layer "B.Cu") (net 6))
+  (segment (start 140.543306 98.216694) (end 145.012528 98.216694) (width 0.25) (layer "B.Cu") (net 5))
+  (segment (start 137.16 101.6) (end 140.543306 98.216694) (width 0.25) (layer "B.Cu") (net 5))
+  (segment (start 145.012528 103.296694) (end 145.012528 104.372528) (width 0.25) (layer "B.Cu") (net 6))
+  (segment (start 145.012528 104.372528) (end 147.32 106.68) (width 0.25) (layer "B.Cu") (net 6))
 )

Commit message: changed circuit
Parts:
- Q1: footprint Package_TO_SOT_THT:TO-92L_Inline_Wide -> Package_TO_SOT_THT:TO-92L_HandSolder
- R3: value 10 -> 10k
- moved Q1 0.78 mm to (145.0, 99.0)
Routing:
- net Net-(D3-Pad2): track 4.34 -> 6.10 mm
Changed lines of the file:
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@@
     )
   )
-  (footprint "Package_TO_SOT_THT:TO-92L_Inline_Wide" (layer "F.Cu")
-    (at 145.012528 98.216694 -90)
-    (descr "TO-92L leads in-line (large body variant of TO-92), also known as TO-226, wide, drill 0.75mm (see https://www.diodes.com/assets/Package-Files/TO92L.pdf and http://www.ti.com/lit/an/snoa059/snoa059.pdf)")
-    (tags "TO-92L Inline Wide transistor")
-    (property "Sheetfile" "light_gate.kicad_sch")
-    (property "Sheetname" "")
-    (attr through_hole)
-    (fp_text reference "Q1" (at 2.54 -3.56 -90) (layer "F.SilkS")
-      (effects (font (size 1 1) (thickness 0.15)))
-    )
-    (fp_text value "BC547" (at 2.54 2.79 -90) (layer "F.Fab")
-      (effects (font (size 1 1) (thickness 0.15)))
-    )
-    (fp_text user "${REFERENCE}" (at 2.54 0 -90) (layer "F.Fab")
-      (effects (font (size 1 1) (thickness 0.15)))
-    )
-    (fp_line (start 0.6 1.7) (end 4.45 1.7) (layer "F.SilkS") (width 0.12))
-    (fp_arc (start 0.1836 -1.098807) (mid 1.143021 -2.192817) (end 2.54 -2.6) (layer "F.SilkS") (width 0.12))
-    (fp_arc (start 2.54 -2.6) (mid 3.936979 -2.192818) (end 4.8964 -1.098807) (layer "F.SilkS") (width 0.12))
-    (fp_arc (start 4.842383 1.112264) (mid 4.666594 1.419753) (end 4.45 1.7) (layer "F.SilkS") (width 0.12))
-    (fp_arc (start 0.6 1.7) (mid 0.389183 1.423933) (end 0.217369 1.122045) (layer "F.SilkS") (width 0.12))
-    (fp_line (start -1 -2.75) (end -1 1.85) (layer "F.CrtYd") (width 0.05))
-    (fp_line (start 6.1 1.85) (end -1 1.85) (layer "F.CrtYd") (width 0.05))
-    (fp_line (start -1 -2.75) (end 6.1 -2.75) (layer "F.CrtYd") (width 0.05))
-    (fp_line (start 6.1 1.85) (end 6.1 -2.75) (layer "F.CrtYd") (width 0.05))
-    (fp_line (start 0.65 1.6) (end 4.4 1.6) (layer "F.Fab") (width 0.1))
-    (fp_arc (start 2.54 -2.48) (mid 4.787211 -1.049019) (end 4.441103 1.592547) (layer "F.Fab") (width 0.1))
-    (fp_arc (start 0.647182 1.602385) (mid 0.290076 -1.043188) (end 2.54 -2.48) (layer "F.Fab") (width 0.1))
-    (pad "1" thru_hole rect (at 0 0 270) (size 1.5 1.5) (drill 0.8) (layers *.Cu *.Mask)
+  (footprint "Package_TO_SOT_THT:TO-92L_HandSolder" (layer "F.Cu")
+    (at 145.012528 99 -90)
+    (descr "TO-92L leads in-line (large body variant of TO-92), also known as TO-226, wide, drill 0.75mm, hand-soldering variant with enlarged pads (see https://www.diodes.com/assets/Package-Files/TO92L.pdf and http://www.ti.com/lit/an/snoa059/snoa059.pdf)")
+    (tags "to-92 sc-43 sc-43a sot54 PA33 transistor")
+    (property "Sheetfile" "light_gate.kicad_sch")
+    (property "Sheetname" "")
+    (attr through_hole)
+    (fp_text reference "Q1" (at 1.27 -3.8 -90) (layer "F.SilkS")
+      (effects (font (size 1 1) (thickness 0.15)))
+    )
+    (fp_text value "BC547" (at 1.27 2.79 -90) (layer "F.Fab")
+      (effects (font (size 1 1) (thickness 0.15)))
+    )
+    (fp_text user "${REFERENCE}" (at 1.27 0 -90) (layer "F.Fab")
+      (effects (font (size 1 1) (thickness 0.15)))
+    )
+    (fp_line (start -0.53 1.85) (end 3.07 1.85) (layer "F.SilkS") (width 0.12))
+    (fp_arc (start -0.541453 1.842156) (mid -1.247298 -0.581475) (end 0.45 -2.45) (layer "F.SilkS") (width 0.12))
+    (fp_arc (start 2.05 -2.45) (mid 3.769931 -0.601036) (end 3.078445 1.827684) (layer "F.SilkS") (width 0.12))
+    (fp_line (start -1.46 -3.05) (end 4 -3.05) (layer "F.CrtYd") (width 0.05))
+    (fp_line (start 4 2.01) (end 4 -3.05) (layer "F.CrtYd") (width 0.05))
+    (fp_line (start -1.45 -3.05) (end -1.46 2.01) (layer "F.CrtYd") (width 0.05))
+    (fp_line (start 4 2.01) (end -1.46 2.01) (layer "F.CrtYd") (width 0.05))
+    (fp_line (start -0.5 1.75) (end 3 1.75) (layer "F.Fab") (width 0.1))
+    (fp_arc (start -0.483625 1.753625) (mid -1.021221 -0.949055) (end 1.27 -2.48) (layer "F.Fab") (width 0.1))
+    (fp_arc (start 1.27 -2.48) (mid 3.561221 -0.949055) (end 3.023625 1.753625) (layer "F.Fab") (width 0.1))
+    (pad "1" thru_hole rect (at 0 0 270) (size 1.1 1.8) (drill 0.75 (offset 0 0.4)) (layers *.Cu *.Mask)
       (net 5 "Net-(Q1-Pad1)") (pinfunction "C") (pintype "passive"))
-    (pad "2" thru_hole circle (at 2.54 0 270) (size 1.5 1.5) (drill 0.8) (layers *.Cu *.Mask)
+    (pad "2" thru_hole roundrect (at 1.27 -1.27 270) (size 1.1 1.8) (drill 0.75 (offset 0 -0.4)) (layers *.Cu *.Mask) (roundrect_rratio 0.25)
       (net 3 "Net-(D2-Pad2)") (pinfunction "B") (pintype "input"))
-    (pad "3" thru_hole circle (at 5.08 0 270) (size 1.5 1.5) (drill 0.8) (layers *.Cu *.Mask)
+    (pad "3" thru_hole roundrect (at 2.54 0 270) (size 1.1 1.8) (drill 0.75 (offset 0 0.4)) (layers *.Cu *.Mask) (roundrect_rratio 0.25)
       (net 6 "Net-(D3-Pad2)") (pinfunction "E") (pintype "passive"))
-    (model "${KICAD6_3DMODEL_DIR}/Package_TO_SOT_THT.3dshapes/TO-92L_Inline_Wide.wrl"
+    (model "${KICAD6_3DMODEL_DIR}/Package_TO_SOT_THT.3dshapes/TO-92L.wrl"
       (offset (xyz 0 0 0))
       (scale (xyz 1 1 1))
@@
       (effects (font (size 1 1) (thickness 0.15)))
     )
-    (fp_text value "10" (at 3.81 2.37 -90) (layer "F.SilkS")
+    (fp_text value "10k" (at 3.81 2.37 -90) (layer "F.SilkS")
       (effects (font (size 1 1) (thickness 0.15)))
     )
@@
   (segment (start 125.73 101.6) (end 127 102.87) (width 0.25) (layer "B.Cu") (net 2))
   (segment (start 127 102.87) (end 127 106.68) (width 0.25) (layer "B.Cu") (net 2))
+  (segment (start 143.57 100.27) (end 146.282528 100.27) (width 0.25) (layer "B.Cu") (net 3))
+  (segment (start 121.92 99.06) (end 129.54 99.06) (width 0.25) (layer "B.Cu") (net 3))
+  (segment (start 129.54 99.06) (end 129.54 104.14) (width 0.25) (layer "B.Cu") (net 3))
   (segment (start 121.92 101.6) (end 121.92 99.06) (width 0.25) (layer "B.Cu") (net 3))
-  (segment (start 139.7 101.6) (end 140.543306 100.756694) (width 0.25) (layer "B.Cu") (net 3))
+  (segment (start 132.08 101.6) (end 132.08 106.68) (width 0.25) (layer "B.Cu") (net 3))
   (segment (start 118.675 101.585) (end 121.905 101.585) (width 0.25) (layer "B.Cu") (net 3))
-  (segment (start 132.08 101.6) (end 132.08 106.68) (width 0.25) (layer "B.Cu") (net 3))
-  (segment (start 129.54 99.06) (end 129.54 104.14) (width 0.25) (layer "B.Cu") (net 3))
   (segment (start 121.905 101.585) (end 121.92 101.6) (width 0.25) (layer "B.Cu") (net 3))
-  (segment (start 121.92 99.06) (end 129.54 99.06) (width 0.25) (layer "B.Cu") (net 3))
+  (segment (start 139.7 104.14) (end 143.57 100.27) (width 0.25) (layer "B.Cu") (net 3))
+  (segment (start 129.54 104.14) (end 139.7 104.14) (width 0.25) (layer "B.Cu") (net 3))
   (segment (start 132.08 106.68) (end 137.16 106.68) (width 0.25) (layer "B.Cu") (net 3))
-  (segment (start 139.7 104.14) (end 139.7 101.6) (width 0.25) (layer "B.Cu") (net 3))
-  (segment (start 140.543306 100.756694) (end 145.012528 100.756694) (width 0.25) (layer "B.Cu") (net 3))
-  (segment (start 129.54 104.14) (end 139.7 104.14) (width 0.25) (layer "B.Cu") (net 3))
   (segment (start 132.08 93.98) (end 137.16 93.98) (width 0.25) (layer "B.Cu") (net 4))
   (segment (start 119.38 93.98) (end 125.73 93.98) (width 0.25) (layer "B.Cu") (net 4))
@@
   (segment (start 142.24 93.98) (end 137.16 93.98) (width 0.25) (layer "B.Cu") (net 4))
   (segment (start 118.675 99.045) (end 118.675 94.685) (width 0.25) (layer "B.Cu") (net 4))
-  (segment (start 140.543306 98.216694) (end 145.012528 98.216694) (width 0.25) (layer "B.Cu") (net 5))
-  (segment (start 137.16 101.6) (end 140.543306 98.216694) (width 0.25) (layer "B.Cu") (net 5))
-  (segment (start 145.012528 103.296694) (end 145.012528 104.372528) (width 0.25) (layer "B.Cu") (net 6))
-  (segment (start 145.012528 104.372528) (end 147.32 106.68) (width 0.25) (layer "B.Cu") (net 6))
+  (segment (start 139 99) (end 139 99.76) (width 0.25) (layer "B.Cu") (net 5))
+  (segment (start 145.012528 99) (end 139 99) (width 0.25) (layer "B.Cu") (net 5))
+  (segment (start 139 99.76) (end 137.16 101.6) (width 0.25) (layer "B.Cu") (net 5))
+  (segment (start 145.012528 101.54) (end 147.32 103.847472) (width 0.25) (layer "B.Cu") (net 6))
+  (segment (start 147.32 103.847472) (end 147.32 106.68) (width 0.25) (layer "B.Cu") (net 6))
 )
