File: Circuits/Magnet_v2/Magnet_v2.kicad_sch (KiCad schematic)
At the start: 10 parts, among them J1 Conn_01x03_Male, Q1 BC547, SW1 -

Commit message: added lm393 to lightgate
Parts:
- R1, R2: footprint (none) -> Resistor_THT:R_Axial_DIN0207_L6.3mm_D2.5mm_P7.62mm_Horizontal
Changed lines of the file:
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@@
   (junction (at 129.54 93.98) (diameter 0) (color 0 0 0 0)
+  )
+  (junction (at 137.16 106.68) (diameter 0) (color 0 0 0 0)
   )
   (junction (at 93.98 106.68) (diameter 0) (color 0 0 0 0)
@@
     (stroke (width 0) (type default) (color 0 0 0 0))
   )
-  (wire (pts (xy 129.54 93.98) (xy 129.54 97.79))
-    (stroke (width 0) (type default) (color 0 0 0 0))
-  )
   (wire (pts (xy 93.98 69.85) (xy 102.87 69.85))
-    (stroke (width 0) (type default) (color 0 0 0 0))
-  )
-  (wire (pts (xy 115.57 106.68) (xy 137.16 106.68))
     (stroke (width 0) (type default) (color 0 0 0 0))
   )
@@
     (stroke (width 0) (type default) (color 0 0 0 0))
   )
+  (wire (pts (xy 129.54 95.25) (xy 129.54 93.98))
+    (stroke (width 0) (type default) (color 0 0 0 0))
+  )
   (wire (pts (xy 137.16 93.98) (xy 129.54 93.98))
+    (stroke (width 0) (type default) (color 0 0 0 0))
+  )
+  (wire (pts (xy 137.16 106.68) (xy 137.16 128.27))
     (stroke (width 0) (type default) (color 0 0 0 0))
   )
@@
     (stroke (width 0) (type default) (color 0 0 0 0))
   )
-  (wire (pts (xy 93.98 106.68) (xy 93.98 110.49))
+  (wire (pts (xy 93.98 106.68) (xy 93.98 129.54))
     (stroke (width 0) (type default) (color 0 0 0 0))
   )
@@
   )
   (wire (pts (xy 123.19 67.31) (xy 129.54 67.31))
+    (stroke (width 0) (type default) (color 0 0 0 0))
+  )
+  (wire (pts (xy 115.57 106.68) (xy 137.16 106.68))
     (stroke (width 0) (type default) (color 0 0 0 0))
   )
@@
     (property "Reference" "R2" (id 0) (at 116.84 78.74 90))
     (property "Value" "47" (id 1) (at 116.84 81.28 90))
-    (property "Footprint" "" (id 2) (at 116.84 86.868 90)
+    (property "Footprint" "Resistor_THT:R_Axial_DIN0207_L6.3mm_D2.5mm_P7.62mm_Horizontal" (id 2) (at 116.84 86.868 90)
       (effects (font (size 1.27 1.27)) hide)
     )
@@
       (effects (font (size 1.27 1.27)) (justify left))
     )
-    (property "Footprint" "" (id 2) (at 107.442 88.9 90)
+    (property "Footprint" "Resistor_THT:R_Axial_DIN0207_L6.3mm_D2.5mm_P7.62mm_Horizontal" (id 2) (at 107.442 88.9 90)
       (effects (font (size 1.27 1.27)) hide)
     )
@@
     (pin "2")
   )
-  (symbol (lib_id "power:VCC") (at 93.98 110.49 180) (unit 1)
+  (symbol (lib_id "power:VCC") (at 93.98 129.54 180) (unit 1)
     (in_bom yes) (on_board yes) (fields_autoplaced)
-    (property "Reference" "#PWR0102" (id 0) (at 93.98 106.68 0)
+    (property "Reference" "#PWR0102" (id 0) (at 93.98 125.73 0)
       (effects (font (size 1.27 1.27)) hide)
     )
-    (property "Value" "VCC" (id 1) (at 93.98 115.57 0))
-    (property "Footprint" "" (id 2) (at 93.98 110.49 0)
+    (property "Value" "VCC" (id 1) (at 93.98 134.62 0))
+    (property "Footprint" "" (id 2) (at 93.98 129.54 0)
       (effects (font (size 1.27 1.27)) hide)
     )
-    (property "Datasheet" "" (id 3) (at 93.98 110.49 0)
+    (property "Datasheet" "" (id 3) (at 93.98 129.54 0)
       (effects (font (size 1.27 1.27)) hide)
     )
@@
     (pin "2")
   )
-  (symbol (lib_id "power:GNDREF") (at 129.54 97.79 0) (unit 1)
+  (symbol (lib_id "power:GNDREF") (at 137.16 128.27 0) (unit 1)
     (in_bom yes) (on_board yes) (fields_autoplaced)
-    (property "Reference" "#PWR0101" (id 0) (at 129.54 104.14 0)
+    (property "Reference" "#PWR0101" (id 0) (at 137.16 134.62 0)
       (effects (font (size 1.27 1.27)) hide)
     )
-    (property "Value" "GNDREF" (id 1) (at 129.54 102.87 0))
-    (property "Footprint" "" (id 2) (at 129.54 97.79 0)
+    (property "Value" "GNDREF" (id 1) (at 137.16 133.35 0))
+    (property "Footprint" "" (id 2) (at 137.16 128.27 0)
       (effects (font (size 1.27 1.27)) hide)
     )
-    (property "Datasheet" "" (id 3) (at 129.54 97.79 0)
+    (property "Datasheet" "" (id 3) (at 137.16 128.27 0)
       (effects (font (size 1.27 1.27)) hide)
     )
