File: Light Gate/Circuits/light_gate_digital/l_g_d/l_g_d/l_g_d.kicad_pcb (KiCad board)
At the start: 2 copper layers, 37 x 25 mm, 14 parts, among them J1 Conn_01x03_Female, U1 LM393P

Commit message: changed resistor
Parts:
- 220: renamed from 1k; value 1k -> 220
Changed lines of the file:
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@@
     (property "Sheetname" "")
     (attr through_hole)
-    (fp_text reference "1k" (at 3.81 0) (layer "F.SilkS")
+    (fp_text reference "220" (at 3.81 0) (layer "F.SilkS")
       (effects (font (size 1 1) (thickness 0.15)))
     )
-    (fp_text value "1k" (at 3.81 2.37) (layer "F.Fab")
+    (fp_text value "220" (at 3.81 2.37) (layer "F.Fab")
       (effects (font (size 1 1) (thickness 0.15)))
     )
