File: Light Gate/Circuits/light_gate_digital/l_g_d_d/l_g_d_d.kicad_pcb (KiCad board)
At the start: 2 copper layers, 61 x 27 mm, 20 parts, among them J1 Conn_01x04_Male, Q1 Q_Photo_NPN_CE, Q2 Q_Photo_NPN_CE, U1 LM393P

Commit message: changed resistor
Parts:
- renumbered 1k to 220
Changed lines of the file:
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@@
     (property "Sheetname" "")
     (attr through_hole)
-    (fp_text reference "1k" (at 3.81 0 90) (layer "F.SilkS")
+    (fp_text reference "220" (at 3.81 0 90) (layer "F.SilkS")
       (effects (font (size 1 1) (thickness 0.15)))
     )
@@
     (property "Sheetname" "")
     (attr through_hole)
-    (fp_text reference "1k" (at 3.81 0.04 90) (layer "F.SilkS")
-      (effects (font (size 1 1) (thickness 0.15)))
-    )
+    (fp_text reference "220" (at 3.81 0.04 90) (layer "F.SilkS")
+      (effects (font (size 1 1) (thickness 0.15)))
+    )
