File: Light Gate/Circuits/light_gate_digital/l_g_d_d/l_g_d_d.kicad_sch (KiCad schematic)
At the start: 17 parts, among them J1 Conn_01x04_Male, Q1 Q_Photo_NPN_CE, Q2 Q_Photo_NPN_CE, U1 LM393P

Commit message: changed resistor
Parts:
- R_IRE2, R_IR_D1: value 1k -> 220
Changed lines of the file:
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@@
       (effects (font (size 1.27 1.27)) (justify left))
     )
-    (property "Value" "1k" (id 1) (at 114.3 110.4899 0)
+    (property "Value" "220" (id 1) (at 114.3 110.4899 0)
       (effects (font (size 1.27 1.27)) (justify left))
     )
@@
       (effects (font (size 1.27 1.27)) (justify left))
     )
-    (property "Value" "1k" (id 1) (at 114.3 74.9299 0)
+    (property "Value" "220" (id 1) (at 114.3 74.9299 0)
       (effects (font (size 1.27 1.27)) (justify left))
     )
@@
     )
     (path "/06451189-3006-498b-bd13-d223f3e85891"
-      (reference "R_IRE2") (unit 1) (value "1k") (footprint "Resistor_THT:R_Axial_DIN0207_L6.3mm_D2.5mm_P7.62mm_Horizontal")
+      (reference "R_IRE2") (unit 1) (value "220") (footprint "Resistor_THT:R_Axial_DIN0207_L6.3mm_D2.5mm_P7.62mm_Horizontal")
     )
     (path "/7fc29542-97f4-4965-90f8-24574a31471b"
@@
     )
     (path "/fbde843f-b9b4-48bb-ab60-be1fb10994a4"
-      (reference "R_IR_D1") (unit 1) (value "1k") (footprint "Resistor_THT:R_Axial_DIN0207_L6.3mm_D2.5mm_P7.62mm_Horizontal")
+      (reference "R_IR_D1") (unit 1) (value "220") (footprint "Resistor_THT:R_Axial_DIN0207_L6.3mm_D2.5mm_P7.62mm_Horizontal")
     )
     (path "/b3908863-1f0b-4105-aa33-a8468a4f004e"
